File: PCB/Main Boards/OSO-SCAN-A1-00 Sensor Candle Concept.brd (EAGLE design)
At the start: 37.1 x 38.1 mm, 58 parts, among them J1 10118193-0001LF, Q1 DMG341, SW2 SPST_TACT-KMR2, U1 AP2112-3.3, U2 ATSAMD11D14A-MUT, U3 LIS2DHTR, U4 AP2112-1.8

Commit message: organize schematic, update some values
Parts:
- LED0, LED1, LED2, LED3, LED6, LED7: value RED -> TBD
- R10, R11, R6, R7, R8, R9: value 2.2K -> TBD
- R3, R4: value 22K -> 10K
