File: PCB/Main Boards/OSO-PYCO-A1-01.brd (EAGLE design)
At the start: 55.9 x 86.4 mm, 71 parts, among them Q1 DMG341, SW1 JS102011SAQN, U1 AP7332-3333W6-7SOT23, U2 MCP73831T-2ACI/OT, U3 ATSAMD51G18A-MUT, U4 2MB Flash, U5 REG710NA-5/3K

Commit message: fix capacitor value
Parts:
- C15: value 2.2uF -> .22uF
Changed lines of the file:
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@@
 <drawing>
 <settings>
-<setting alwaysvectorfont="yes"/>
+<setting alwaysvectorfont="no"/>
 <setting keepoldvectorfont="yes"/>
 <setting verticaltext="up"/>
@@
 <attribute name="VALUE" x="-5.4074" y="4.2716" size="0.508" layer="28" font="vector" ratio="18" rot="MR270" align="center"/>
 </element>
-<element name="C15" library="microbuilder" package="_0603MP" value="2.2uF" x="-10.668" y="4.318" smashed="yes" rot="MR270">
+<element name="C15" library="microbuilder" package="_0603MP" value=".22uF" x="-10.668" y="4.318" smashed="yes" rot="MR270">
 <attribute name="NAME" x="-10.6807" y="2.7686" size="0.508" layer="26" font="vector" ratio="18" rot="MR180" align="center"/>
 <attribute name="REV" value="A" x="-10.668" y="4.318" size="1.778" layer="28" rot="MR270" display="off"/>
