File: PCB/Main Boards/OSO-PYCO-A1-02 (WIP - DO NOT ORDER).brd (EAGLE design)
At the start: 55.9 x 86.4 mm, 71 parts, among them Q1 DMG341, SW1 JS102011SAQN, U1 AP7332-3333W6-7SOT23, U2 MCP73831T-2ACI/OT, U3 ATSAMD51G18A-MUT, U4 2MB Flash, U5 REG710NA-5/3K

Commit message: starting work on pycorder rev 02
Parts:
- moved C4 4.57 mm to (-3.56, 27.7), turned to 180 degrees
- moved C5 4.57 mm to (-8.13, 27.7), turned to 0 degrees
- moved TP1 2.54 mm to (-21.3, 8.38)
- moved TP2 2.54 mm to (-21.3, 10.9)
Connections:
- net +3V3: now also U1.1; no longer U1.6
- net 3.3V: now also U1.6; no longer U1.1
Routing:
- net +3V3: track 102.1 -> 103.8 mm, vias 7 -> 6
