File: PCB/Main Boards/OSO-PYCO-A1-02 (WIP - DO NOT ORDER).sch (EAGLE design)
At the start: 69 parts, among them Q1 DMG341, SW1 JS102011SAQN, U1 AP7332-3333W6-7SOT23, U2 MCP73831T-2ACI/OT, U3 ATSAMD51G18A-MUT, U4 2MB Flash, U5 REG710NA-5/3K

Commit message: starting work on pycorder rev 02
Connections:
- net +3V3: now also U1.OUT2; no longer U1.OUT1
- net 3.3V: now also U1.OUT1; no longer U1.OUT2
Other:
- moved on the sheet: C4, C5
Changed lines of the file:
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@@
 <attribute name="VALUE" x="48.72" y="155.48" size="1.27" layer="96" font="vector" rot="R90"/>
 </instance>
-<instance part="C5" gate="G$1" x="99.06" y="162.56" smashed="yes" rot="R90">
-<attribute name="NAME" x="98.52" y="160.77" size="1.27" layer="95" font="vector" rot="R180"/>
-<attribute name="VALUE" x="98.52" y="165.56" size="1.27" layer="96" font="vector" rot="R180"/>
-</instance>
-<instance part="U$26" gate="G$1" x="101.6" y="160.02" smashed="yes">
-<attribute name="VALUE" x="100.076" y="157.48" size="1.27" layer="96"/>
+<instance part="C5" gate="G$1" x="101.6" y="139.7" smashed="yes" rot="R90">
+<attribute name="NAME" x="101.06" y="137.91" size="1.27" layer="95" font="vector" rot="R180"/>
+<attribute name="VALUE" x="101.06" y="142.7" size="1.27" layer="96" font="vector" rot="R180"/>
+</instance>
+<instance part="U$26" gate="G$1" x="104.14" y="137.16" smashed="yes">
+<attribute name="VALUE" x="102.616" y="134.62" size="1.27" layer="96"/>
 </instance>
 <instance part="U$27" gate="G$1" x="165.1" y="7.62" smashed="yes"/>
@@
 <attribute name="VALUE" x="66.04" y="127" size="1.778" layer="96"/>
 </instance>
-<instance part="+3V3" gate="G$1" x="93.98" y="170.18" smashed="yes" rot="MR0">
-<attribute name="VALUE" x="94.996" y="170.942" size="1.778" layer="96" rot="MR180"/>
+<instance part="+3V3" gate="G$1" x="93.98" y="147.32" smashed="yes" rot="MR0">
+<attribute name="VALUE" x="94.996" y="148.082" size="1.778" layer="96" rot="MR180"/>
 </instance>
 <instance part="GND2" gate="1" x="167.64" y="106.68" smashed="yes">
@@
 <attribute name="VALUE" x="65.7606" y="166.5986" size="2.0828" layer="96" ratio="6" rot="SR0"/>
 </instance>
-<instance part="C4" gate="G$1" x="99.06" y="139.7" smashed="yes" rot="R90">
-<attribute name="NAME" x="98.52" y="137.91" size="1.27" layer="95" font="vector" rot="R180"/>
-<attribute name="VALUE" x="98.52" y="142.7" size="1.27" layer="96" font="vector" rot="R180"/>
-</instance>
-<instance part="U$43" gate="G$1" x="101.6" y="137.16" smashed="yes">
-<attribute name="VALUE" x="100.076" y="134.62" size="1.27" layer="96"/>
-</instance>
-<instance part="U$45" gate="G$1" x="93.98" y="154.94" smashed="yes">
-<attribute name="VALUE" x="92.456" y="155.956" size="1.27" layer="96"/>
+<instance part="C4" gate="G$1" x="101.6" y="162.56" smashed="yes" rot="R90">
+<attribute name="NAME" x="101.06" y="160.77" size="1.27" layer="95" font="vector" rot="R180"/>
+<attribute name="VALUE" x="101.06" y="165.56" size="1.27" layer="96" font="vector" rot="R180"/>
+</instance>
+<instance part="U$43" gate="G$1" x="104.14" y="160.02" smashed="yes">
+<attribute name="VALUE" x="102.616" y="157.48" size="1.27" layer="96"/>
+</instance>
+<instance part="U$45" gate="G$1" x="93.98" y="172.72" smashed="yes">
+<attribute name="VALUE" x="92.456" y="173.736" size="1.27" layer="96"/>
 </instance>
 <instance part="P+3" gate="1" x="45.72" y="170.18" smashed="yes">
@@
 </segment>
 <segment>
-<wire x1="93.98" y1="162.56" x2="93.98" y2="167.64" width="0.1524" layer="91"/>
-<pinref part="C5" gate="G$1" pin="1"/>
-<junction x="93.98" y="162.56"/>
-<pinref part="+3V3" gate="G$1" pin="+3V3"/>
-<pinref part="U1" gate="A" pin="OUT1"/>
-</segment>
-<segment>
 <wire x1="40.64" y1="124.46" x2="43.18" y2="124.46" width="0.1524" layer="91"/>
 <wire x1="43.18" y1="124.46" x2="45.72" y2="124.46" width="0.1524" layer="91"/>
@@
 <pinref part="+3V1" gate="G$1" pin="+3V3"/>
 <junction x="43.18" y="124.46"/>
+</segment>
+<segment>
+<pinref part="U1" gate="A" pin="OUT2"/>
+<pinref part="C5" gate="G$1" pin="1"/>
+<wire x1="93.98" y1="139.7" x2="96.52" y2="139.7" width="0.1524" layer="91"/>
+<pinref part="+3V3" gate="G$1" pin="+3V3"/>
+<wire x1="93.98" y1="139.7" x2="93.98" y2="144.78" width="0.1524" layer="91"/>
+<junction x="93.98" y="139.7"/>
 </segment>
 </net>
@@
 </net>
 <net name="3.3V" class="1">
-<segment>
-<pinref part="U1" gate="A" pin="OUT2"/>
-<pinref part="C4" gate="G$1" pin="1"/>
-<wire x1="93.98" y1="139.7" x2="93.98" y2="152.4" width="0.1524" layer="91"/>
-<junction x="93.98" y="139.7"/>
-<pinref part="U$45" gate="G$1" pin="3.3V"/>
-</segment>
 <segment>
 <wire x1="121.92" y1="157.48" x2="124.46" y2="157.48" width="0.1524" layer="91"/>
@@
 <pinref part="U$65" gate="G$1" pin="3.3V"/>
 </segment>
-</net>
+<segment>
+<pinref part="U$45" gate="G$1" pin="3.3V"/>
+<pinref part="U1" gate="A" pin="OUT1"/>
+<wire x1="93.98" y1="170.18" x2="93.98" y2="162.56" width="0.1524" layer="91"/>
+<pinref part="C4" gate="G$1" pin="1"/>
+<wire x1="93.98" y1="162.56" x2="96.52" y2="162.56" width="0.1524" layer="91"/>
+<junction x="93.98" y="162.56"/>
+</segment>
+</net>
