File: PCB/Main Boards/OSO-SWAT-A1-0x.brd (EAGLE design)
At the start: 24.4 x 24.4 mm, 25 parts, among them J1 FH19C-9S-0.5SH_10_, U1 ATSAML22G18A-MUT

Commit message: watch stuff
Parts:
- removed L2: 10uH, Adafruit 3.5in 480x320 FeatherWing:MICROBUILDER__0805MP
- removed Q2: (no value), Adafruit MONSTER M4SK:SOT23-R
- removed RESET: EVP-BB1AAB000, EVP-BB1AAB000:SW_EVP-BB1AAB000
- added BOOT: EVP-BB1AAB000, EVP-BB1AAB000:SW_EVP-BB1AAB000
- added GND, RST, V+: (no value), Adafruit Feather M0 Express:MICROBUILDER_TESTPOINT_PAD_1MM
- added R5, R6: 1K, microbuilder:_0603MP
- added U2: MIC5365-3.3YC5-TR, MIC5365-3.3YC5-TR:SOT65P210X110-5N
- C1: value 10uF -> 0.1uF
- C4: value 0.1uF -> 10uF
- R2: value 1K -> 10K; device microbuilder:_0603MP -> microbuilder:_0402MP
- moved D1 19.5 mm to (10.0, 0.94), turned to 0 degrees
- moved R2 16.2 mm to (6.22, -9.78)
- moved SWD 10.1 mm to (6.50, -10.0), flipped to the bottom
- moved C5 5.10 mm to (-3.32, 4.19), turned to 135 degrees
- moved C4 3.23 mm to (11.4, -0.79), turned to 270 degrees
- moved LED 0.99 mm to (-11.4, -0.25)
- moved SWC 0.46 mm to (-11.3, -1.27), flipped to the bottom
- moved C7 0.13 mm to (7.16, -5.92)
- moved X1 0.13 mm to (7.37, -3.53)
Connections:
- removed net D0: J1.4, U1.37
- removed net D1: J1.3, U1.38
- removed net N$2: D1.C, Q2.3
- removed net SWCLK/MODE_BTN: R1.2, SWC.P$1, U$2.MODE, U1.45
- removed net SWDIO/SET_BTN: SWD.P$1, U$2.ALARM, U1.46
- new net 3.3V: D1.A, U2.5
- new net D0/MODE: J1.4, U$2.MODE, U1.37
- new net D1/ALARM: BOOT.B1, BOOT.B2, J1.3, U$2.ALARM, U1.38
- new net SWCLK: R1.2, SWC.P$1, U1.45
- new net SWDIO: SWD.P$1, U1.46
- net !RESET: now also R2.2, RST.P$1; no longer RESET.B1, RESET.B2
- net BUZZER: now also R6.1; no longer Q2.1
- net BUZZER_OUT: now also R6.2; no longer D1.A, L2.2
- net COM0: now also U1.7; no longer U1.24
- net COM1: now also U1.8; no longer U1.23
- net COM2: now also U1.9; no longer U1.22
- net GND: now also BOOT.A1, BOOT.A2, GND.P$1, U2.2; no longer Q2.2, RESET.A1, RESET.A2
- net LED/LIGHT_BTN: now also R5.2; no longer R2.2
- net N$1: now also R5.1; no longer R2.1
- net SEG0: now also U1.22; no longer U1.16
- net SEG10: now also U1.10; no longer U1.7
- net SEG2: now also U1.21; no longer U1.15
- net SEG22: now also U1.24; no longer U1.21
- net SEG23: now also U1.23; no longer U1.20
- net SEG3: now also U1.20; no longer U1.14
- net SEG4: now also U1.16; no longer U1.13
- net SEG5: now also U1.15; no longer U1.12
- net SEG6: now also U1.14; no longer U1.11
- net SEG7: now also U1.13; no longer U1.10
- net SEG8: now also U1.12; no longer U1.9
- net SEG9: now also U1.11; no longer U1.8
- net VBUS: now also U2.1, U2.3
- net VCC: now also D1.C, R2.1, V+.P$1; no longer L2.1
Routing:
- net SWCLK/MODE_BTN: track 26.0 -> 0.00 mm, vias 2 -> 0
- net SWCLK: track 0.00 -> 24.9 mm, vias 0 -> 3
- net D1/ALARM: track 0.00 -> 22.9 mm, vias 0 -> 3
- net D0/MODE: track 0.00 -> 22.0 mm, vias 0 -> 3
- net VBUS: track 0.00 -> 19.9 mm, vias 0 -> 2
- net SWDIO/SET_BTN: track 15.0 -> 0.00 mm, vias 1 -> 0
- net COM0: track 5.22 -> 18.9 mm, vias 0 -> 2
- net SWDIO: track 0.00 -> 11.6 mm, vias 0 -> 3
- net COM1: track 5.32 -> 16.4 mm, vias 0 -> 2
- net D0: track 9.95 -> 0.00 mm, vias 2 -> 0
- net D1: track 9.64 -> 0.00 mm, vias 2 -> 0
- net COM2: track 5.16 -> 13.7 mm, vias 0 -> 2
- net VCC: track 69.3 -> 77.5 mm
- net VLCD: track 1.36 -> 5.10 mm, vias 0 -> 2
- net 3.3V: track 0.00 -> 3.73 mm, vias 0 -> 2
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Other:
- board text added: "5V D- D+ NC GND"
- board text added: "9-pin connector: A0: PA02/I2 SDA: PA22/SERCOM2 SCL: PA23/SERCOM2 A1: PB03/I3/TC2[1] A2: PB02/I2/TC2[0] D0: PB22/I6/TC3[0] D1: PB23/I7/TC3[1]"
- board text added: "A watch mod for the Casio F-91W, based on Pluto by CarrotIndustries, arm-watch by @GregDavill and GoodWatch by @travisgoodspeed. CC-BY-SA 4.0, except the bear."
- board text added: "Alarm PB22/I6"
- board text added: "IMPORTANT:"
- board text added: "Mode PB23/I7"
- board text added: "OSO-SWAT-A1-0x"
- board text added: "PB23"
- board text added: "REMOVE BATTERY BEFORE USING USB!!!"
- board text added: "USB D- PA24 D+ PA25"
- board text removed: "9-pin connector: A0: PA02/I2 SDA: PA22/SERCOM2 SCL: PA23/SERCOM2 A1: PB03/I3/TC2[1] A2: PB02/I2/TC2[0] D1: PB22/I6/TC3[0] D2: PB23/I7/TC3[1]"
- board text removed: "A watch mod for the Casio F-91W. Based on arm-watch by @GregDavill, GoodWatch by @travisgoodspeed, and Pluto by CarrotIndustries. CC-BY-SA 4.0, except the bear."
- board text removed: "Alarm Btn: PA31/I11"
- board text removed: "Mode Button: PA30/I10 Has external pull-up."
- board text removed: "NC D- D+ NC GND"
- board text removed: "OSO-SWAT-A1-00"
- board text removed: "USB D- PA24 D+ PA25 VBUS is NC"
