File: PCB/Main Boards/OSO-SWAT-A1-0x.sch (EAGLE design)
At the start: 23 parts, among them J1 FH19C-9S-0.5SH_10_, U1 ATSAML22G18A-MUT

Commit message: watch stuff
Parts:
- removed L2: 10uH, Adafruit 3.5in 480x320 FeatherWing:MICROBUILDER_INDUCTOR_0805MP
- removed Q2: (no value), Adafruit MONSTER M4SK:MOSFET-NREFLOW
- removed RESET: EVP-BB1AAB000, EVP-BB1AAB000:EVP-BB1AAB000
- added BOOT: EVP-BB1AAB000, EVP-BB1AAB000:EVP-BB1AAB000
- added GND, RST, V+: (no value), Adafruit Feather M0 Express:MICROBUILDER_TESTPOINTPAD1MM
- added R5, R6: 1K, microbuilder:RESISTOR_0603MP
- added U2: MIC5365-3.3YC5-TR, MIC5365-3.3YC5-TR:MIC5365-3.3YC5-TR
- C1: value 10uF -> 0.1uF
- C4: value 0.1uF -> 10uF
- R2: value 1K -> 10K; device microbuilder:RESISTOR_0603MP -> microbuilder:RESISTOR_0402MP
Connections:
- removed net D0: J1.4, U1A.PB22/I6/SERCOM0.2
- removed net D1: J1.3, U1A.PB23/I7/SERCOM0.3
- removed net N$2: D1.C, Q2.D
- removed net SWCLK/MODE_BTN: R1.2, SWC.P$1, U$2G$2.MODE, U1A.PA30/I10/SERCOM1.2/SWCLK
- removed net SWDIO/SET_BTN: SWD.P$1, U$2G$2.ALARM, U1A.PA31/I11/SERCOM1.3/SWDIO
- new net 3.3V: D1.A, U2.VOUT
- new net D0/MODE: J1.4, U$2G$2.MODE, U1A.PB22/I6/SERCOM0.2
- new net D1/ALARM: BOOT.B1, BOOT.B2, J1.3, U$2G$2.ALARM, U1A.PB23/I7/SERCOM0.3
- new net SWCLK: R1.2, SWC.P$1, U1A.PA30/I10/SERCOM1.2/SWCLK
- new net SWDIO: SWD.P$1, U1A.PA31/I11/SERCOM1.3/SWDIO
- new net VBUS: U$2G$4.VBUS, U2.EN, U2.VIN
- net !RESET: now also R2.2, RST.P$1; no longer RESET.B1, RESET.B2
- net BUZZER: now also R6.1; no longer Q2.G
- net BUZZER_OUT: now also R6.2; no longer D1.A, L2.2
- net COM0: now also U1A.PB08/I8/AIN2/SERCOM3.0/SLCD[2]; no longer U1A.PA15/I15/SERCOM3.3/SLCD[31]
- net COM1: now also U1A.PB09/I9/AIN3/SERCOM3.1/SLCD[3]; no longer U1A.PA14/I14/SERCOM3.2/SLCD[30]
- net COM2: now also U1A.PA04/I4/AIN4/SERCOM0.0/SLCD[4]; no longer U1A.PA13/I13/SERCOM3.1(I2C)/SLCD[29]
- net GND: now also BOOT.A1, BOOT.A2, GND.P$1, U2.GND; no longer Q2.S, RESET.A1, RESET.A2
- net LED/LIGHT_BTN: now also R5.2; no longer R2.2
- net N$1: now also R5.1; no longer R2.1
- net SEG0: now also U1A.PA13/I13/SERCOM3.1(I2C)/SLCD[29]; no longer U1A.PA11/I11/SERCOM0.3/SLCD[14]
- net SEG10: now also U1A.PA05/I5/AIN5/SERCOM0.1/SLCD[5]; no longer U1A.PB08/I8/AIN2/SERCOM3.0/SLCD[2]
- net SEG2: now also U1A.PA12/I12/SERCOM3.0(I2C)/SLCD[28]; no longer U1A.PA10/I10/SERCOM0.2/SLCD[13]
- net SEG22: now also U1A.PA15/I15/SERCOM3.3/SLCD[31]; no longer U1A.PA12/I12/SERCOM3.0(I2C)/SLCD[28]
- net SEG23: now also U1A.PA14/I14/SERCOM3.2/SLCD[30]; no longer U1A.PB11/SERCOM3.3/SLCD[21]
- net SEG3: now also U1A.PB11/SERCOM3.3/SLCD[21]; no longer U1A.PA09/I9/SERCOM0.1/SLCD[12]
- net SEG4: now also U1A.PA11/I11/SERCOM0.3/SLCD[14]; no longer U1A.PA08/NMI/SERCOM0.0/SLCD[11]
- net SEG5: now also U1A.PA10/I10/SERCOM0.2/SLCD[13]; no longer U1A.PA07/I7/AIN7/SERCOM0.3/SLCD[7]
- net SEG6: now also U1A.PA09/I9/SERCOM0.1/SLCD[12]; no longer U1A.PA06/I6/AIN6/SERCOM0.2/SLCD[6]
- net SEG7: now also U1A.PA08/NMI/SERCOM0.0/SLCD[11]; no longer U1A.PA05/I5/AIN5/SERCOM0.1/SLCD[5]
- net SEG8: now also U1A.PA07/I7/AIN7/SERCOM0.3/SLCD[7]; no longer U1A.PA04/I4/AIN4/SERCOM0.0/SLCD[4]
- net SEG9: now also U1A.PA06/I6/AIN6/SERCOM0.2/SLCD[6]; no longer U1A.PB09/I9/AIN3/SERCOM3.1/SLCD[3]
- net VCC: now also D1.C, R2.1, V+.P$1; no longer L2.1
Other:
- moved on the sheet: D1, R2, U$2G$1, U$2G$2, U$2G$4
