File: PCB/Main Boards/OSO-SWAT-A1-0xA.sch (EAGLE design)
At the start: 23 parts, among them J1 FH19C-9S-0.5SH_10_, U1 ATSAML22G18A-MUT

Commit message: watch stuff
Parts:
- removed D1: SCHOTTKY, adafruit:DIODESOD-323F
- removed L2: 10uH, Adafruit 3.5in 480x320 FeatherWing:MICROBUILDER_INDUCTOR_0805MP
- removed Q2: (no value), Adafruit MONSTER M4SK:MOSFET-NREFLOW
- removed U1: ATSAML22G18A-MUT, ATSAML22G18A-MUT:ATSAML22G18A-MUT
- added GND, RST, V+: (no value), Adafruit Feather M0 Express:MICROBUILDER_TESTPOINTPAD1MM
- added R5: 10K, microbuilder:RESISTOR_0603MP
- added R6: 1K, microbuilder:RESISTOR_0603MP
- added U2: ATSAML22J18A-MUT, ATSAML22:ATSAML22J18A-MUT
Connections:
- removed net D0: J1.4, U1A.PB22/I6/SERCOM0.2
- removed net D1: J1.3, U1A.PB23/I7/SERCOM0.3
- removed net N$2: D1.C, Q2.D
- removed net SWCLK/MODE_BTN: R1.2, SWC.P$1, U$2G$2.MODE, U1A.PA30/I10/SERCOM1.2/SWCLK
- removed net SWDIO/SET_BTN: SWD.P$1, U$2G$2.ALARM, U1A.PA31/I11/SERCOM1.3/SWDIO
- new net ALARM: U$2G$2.ALARM
- new net D0_CS: J1.4
- new net D1_MISO: J1.3, RESET.B1, RESET.B2
- new net MODE: U$2G$2.MODE
- new net SWCLK: R1.2, SWC.P$1
- net !RESET: now also R5.2, RST.P$1; no longer RESET.B1, RESET.B2, U1A.RESET
- net A0: no longer U1A.PA02/I2/AIN0
- net A1_SCK: no longer U1A.PB03/I3/AIN11/SERCOM3.1
- net A2_MOSI: no longer U1A.PB02/I2/AIN10/SERCOM3.0
- net BUZZER: now also R6.2; no longer Q2.G, U1A.PA27/I15
- net BUZZER_OUT: now also R6.1; no longer D1.A, L2.2
- net COM0: now also U2A.PB06/I6/AIN14/SLCD[0]; no longer U1A.PA15/I15/SERCOM3.3/SLCD[31]
- net COM1: now also U2A.PB07/I7/AIN15/SLCD[1]; no longer U1A.PA14/I14/SERCOM3.2/SLCD[30]
- net COM2: now also U2A.PB08/I8/AIN2/SERCOM3.0/SLCD[2]; no longer U1A.PA13/I13/SERCOM3.1(I2C)/SLCD[29]
- net GND: now also GND.P$1; no longer Q2.S, U1B.EPAD, U1B.GND, U1B.GNDANA, U1B.GND_2, U1B.GND_3
- net LED/LIGHT_BTN: no longer U1A.PA03/I3/AIN1
- net SCL: no longer U1A.PA23/I7/SERCOM0.3+2.1(I2C)/SLCD[51]
- net SDA: no longer U1A.PA22/I6/SERCOM0.2+2.0(I2C)/SLCD[50]
- net SEG0: now also U2A.PB12/I12/SERCOM3.0/SLCD[22]; no longer U1A.PA11/I11/SERCOM0.3/SLCD[14]
- net SEG1: now also U2A.PB11/I11/SERCOM3.3/SLCD[21]
- net SEG10: now also U2A.PB09/I9/AIN3/SERCOM3.1/SLCD[3]; no longer U1A.PB08/I8/AIN2/SERCOM3.0/SLCD[2]
- net SEG16: no longer U1A.PA21/I5/SERCOM0.1+2.3/SLCD[49]
- net SEG17: no longer U1A.PA20/I4/SERCOM0.0+2.2/SLCD[48]
- net SEG18: no longer U1A.PA19/I3/SERCOM1+2.3/SLCD[35]
- net SEG19: no longer U1A.PA18/I2/SERCOM1+2.2/SLCD[34]
- net SEG2: now also U2A.PA11/I11/SERCOM0.3/SLCD[14]; no longer U1A.PA10/I10/SERCOM0.2/SLCD[13]
- net SEG20: no longer U1A.PA17/I1/SERCOM1+2.1/SLCD[33]
- net SEG21: no longer U1A.PA16/I0/SERCOM1+2.0/SLCD[32]
- net SEG22: no longer U1A.PA12/I12/SERCOM3.0(I2C)/SLCD[28]
- net SEG23: no longer U1A.PB11/SERCOM3.3/SLCD[21]
- net SEG26: now also U2A.PB15/I15/SERCOM3.3/SLCD[25]
- net SEG27: now also U2A.PB14/I14/SERCOM3.2/SLCD[24]
- net SEG28: now also U2A.PB13/SERCOM3.1/SLCD[23]
- net SEG3: now also U2A.PA10/I10/SERCOM0.2/SLCD[13]; no longer U1A.PA09/I9/SERCOM0.1/SLCD[12]
- net SEG4: now also U2A.PA09/I9/SERCOM0.1/SLCD[12]; no longer U1A.PA08/NMI/SERCOM0.0/SLCD[11]
- net SEG5: now also U2A.PA08/NMI/SERCOM0.0/SLCD[11]; no longer U1A.PA07/I7/AIN7/SERCOM0.3/SLCD[7]
- net SEG6: now also U2A.PA07/I7/AIN7/SERCOM0.3/SLCD[7]; no longer U1A.PA06/I6/AIN6/SERCOM0.2/SLCD[6]
- net SEG7: now also U2A.PA06/I6/AIN6/SERCOM0.2/SLCD[6]; no longer U1A.PA05/I5/AIN5/SERCOM0.1/SLCD[5]
- net SEG8: now also U2A.PA05/I5/AIN5/SERCOM0.1/SLCD[5]; no longer U1A.PA04/I4/AIN4/SERCOM0.0/SLCD[4]
- net SEG9: now also U2A.PA04/I4/AIN4/SERCOM0.0/SLCD[4]; no longer U1A.PB09/I9/AIN3/SERCOM3.1/SLCD[3]
- net USB_N: no longer U1A.PA24/I12/SERCOM2.2/USB-
- net USB_P: no longer U1A.PA25/I13/SERCOM2.3/USB+
- net VCC: now also R5.1, V+.P$1; no longer L2.1, U1B.VDDANA, U1B.VDDIO, U1B.VDDIO_2, U1B.VDDIO_3
- net VDDCORE: no longer U1B.VDDCORE
- net VDDOUT: no longer U1B.VDDOUT
- net VLCD: no longer U1B.VLCD
- net XIN32: no longer U1A.PA00/XIN32/EXTINT[0]/SERCOM1.0
- net XOUT32: no longer U1A.PA01/XOUT32/EXTINT[1]/SERCOM1.1
Other:
- moved on the sheet: C6, C7, RESET, X1
