File: PCB/Main Boards/OSO-PYCO-A1-02.brd (EAGLE design)
At the start: 55.9 x 86.4 mm, 71 parts, among them Q1 DMG341, SW1 JS102011SAQN, U1 AP7332-3333W6-7SOT23, U2 MCP73831T-2ACI/OT, U3 ATSAMD51G18A-MUT, U4 2MB Flash, U5 REG710NA-5/3K

Commit message: new pycorder and sensor watch
Parts:
- removed R15, R16: 1M, EXB2HV470JV:EXB2HV
- removed U$32: MATRIX_PASSIVE_8X4SEG, My Stuff:MATRIX_ACTIVE_8X4SEG_4MM
- added B1, B2: EVQQ, microbuilder:6MMX6MM_TACTILE_SMT
- added U$24: K1-5202UA, K1-5202UA:K1-5202UA
- moved C12 7.37 mm to (-3.30, -26.7)
- moved D2 7.37 mm to (15.0, 21.3)
- moved R10 7.37 mm to (-7.87, -26.7)
- moved R11 7.37 mm to (-12.7, 27.4)
- moved R12 7.37 mm to (-15.5, 27.4)
- moved SW1 7.37 mm to (26.1, 25.2)
- moved C17 7.37 mm to (-12.5, 8.00)
- moved R6 7.37 mm to (26.2, -20.6)
- moved C9 7.37 mm to (-19.8, -12.8)
- moved FFC 7.37 mm to (-16.3, 3.56)
- moved TP2 7.37 mm to (-21.3, 3.56)
- moved 9-PIN-CONNECTOR 7.37 mm to (-25.4, -9.65)
- moved BATTERY 7.37 mm to (10.9, -24.1)
- moved C1 7.37 mm to (9.40, 22.9)
- moved C10 7.37 mm to (-7.34, -19.6)
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Connections:
- removed net SWCLK/DISP: C18.1, FFC.P$5, R14.1, TP3.P$1, U3.45
- removed net SWDIO/EXTCOMIN: FFC.P$4, TP6.P$1, U3.46
- removed net X0: R16.9, U$32.X0Y0, U$32.X0Y1, U$32.X0Y2, U$32.X0Y3, U$32.X0Y4, U3.30
- removed net X1: R16.14, U$32.X1Y0, U$32.X1Y1, U$32.X1Y2, U$32.X1Y3, U$32.X1Y4, U3.28
- removed net X2: R16.15, U$32.X2Y0, U$32.X2Y1, U$32.X2Y2, U$32.X2Y3, U$32.X2Y4, U3.27
- removed net X3: R16.16, U$32.X3Y0, U$32.X3Y1, U$32.X3Y2, U$32.X3Y3, U$32.X3Y4, U3.26
- removed net X4: R15.16, U$32.X4Y0, U$32.X4Y1, U$32.X4Y2, U$32.X4Y3, U$32.X4Y4, U3.25
- removed net X5: R15.15, U$32.X5Y0, U$32.X5Y1, U$32.X5Y2, U$32.X5Y3, U$32.X5Y4, U3.24
- removed net X6: R15.14, U$32.X6Y0, U$32.X6Y1, U$32.X6Y2, U$32.X6Y3, U$32.X6Y4, U3.23
- removed net X7: R15.9, U$32.X7Y0, U$32.X7Y1, U$32.X7Y2, U$32.X7Y3, U$32.X7Y4, U3.1
- removed net X8: R15.10, U$32.X8Y0, U$32.X8Y1, U$32.X8Y2, U$32.X8Y3, U$32.X8Y4, U3.2
- removed net X9: R15.11, U$32.X9Y0, U$32.X9Y1, U$32.X9Y2, U$32.X9Y3, U$32.X9Y4, U3.4
- removed net Y0: R16.10, U$32.Y0X0, U$32.Y0X1, U$32.Y0X10, U$32.Y0X2, U$32.Y0X3, U$32.Y0X4, U$32.Y0X5, U$32.Y0X6, U$32.Y0X7, U$32.Y0X8, U$32.Y0X9, U3.29
- removed net Y1: R16.11, U$32.Y1X0, U$32.Y1X1, U$32.Y1X10, U$32.Y1X2, U$32.Y1X3, U$32.Y1X4, U$32.Y1X5, U$32.Y1X6, U$32.Y1X7, U$32.Y1X8, U$32.Y1X9, U3.31
- removed net Y2: R16.12, U$32.Y2X0, U$32.Y2X1, U$32.Y2X10, U$32.Y2X2, U$32.Y2X3, U$32.Y2X4, U$32.Y2X5, U$32.Y2X6, U$32.Y2X7, U$32.Y2X8, U$32.Y2X9, U3.32
- removed net Y3: R16.13, U$32.Y3X0, U$32.Y3X1, U$32.Y3X10, U$32.Y3X2, U$32.Y3X3, U$32.Y3X4, U$32.Y3X5, U$32.Y3X6, U$32.Y3X7, U$32.Y3X8, U$32.Y3X9, U3.39
- new net CENTER: U$24.P$2, U3.27
- new net DISP: C18.1, FFC.P$5, R14.1, U3.1
- new net EXTCOMIN: FFC.P$4, U3.2
- new net NE: U$24.P$4, U3.25
- new net NEXT: B2.B, U3.24
- new net NW: U$24.P$1, U3.26
- new net PREV: B1.B', U3.30
- new net SE: U$24.P$6, U3.29
- new net SW: U$24.P$3, U3.28
- new net SWCLK: TP3.P$1, U3.45
- new net SWDIO: TP6.P$1, U3.46
- net 3.3V: now also U3.4; no longer R14.2
- net GND: now also B1.A, B1.A', B2.A, B2.A', R14.2, U$24.P$5, U$24.P$7, U$24.P$8; no longer R15.1, R15.2, R15.3, R15.4, R15.5, R15.6, R15.7, R15.8, R16.1, R16.2, R16.3, R16.4, R16.5, R16.6, R16.7, R16.8
Routing:
- net X7: track 101.3 -> 0.00 mm
- net X5: track 96.4 -> 0.00 mm
- net X8: track 94.4 -> 0.00 mm
- net X6: track 92.7 -> 0.00 mm
- net X9: track 87.9 -> 0.00 mm
- net Y3: track 81.7 -> 0.00 mm
- net Y2: track 72.7 -> 0.00 mm
- net X4: track 72.6 -> 0.00 mm
- net Y1: track 71.6 -> 0.00 mm
- net Y0: track 65.6 -> 0.00 mm
- net X3: track 61.4 -> 0.00 mm
- net X2: track 54.1 -> 0.00 mm
- net GND: track 150.3 -> 201.2 mm, vias 26 -> 37
- net X1: track 47.0 -> 0.00 mm
- net SWCLK/DISP: track 43.4 -> 0.00 mm, vias 4 -> 0
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Other:
- board size 55.9 x 86.4 mm -> 55.9 x 80.8 mm
- board text added: "JLCJLCJLC"
- board text added: "OSO-PYCO-A1-02"
- board text added: "RST"
- board text added: "by Joey Castillo / @josecastillo. Includes elements of @Adafruit's Sharp Memory Display Breakout. Looks best in @OSHPark After Dark. Crafted with in Brooklyn, NY. Lazer bear by @DoctorDevens. plz don't steal the bear =)"
- board text removed: "OSO-PYCO-A1-01"
- board text removed: "RESET"
- board text removed: "by Joey Castillo / @josecastillo. Includes elements of @Adafruit's Sharp Memory Display Breakout, and a touch matrix inspired by @PatternAgents' awesome library of touch widgets. Boards by @OSHPark (After Dark). Crafted with in Brooklyn, NY. Lazer bear by @DoctorDevens. plz don't steal the bear =)"
