File: PCB/Main Boards/OSO-PYCO-A1-02.sch (EAGLE design)
At the start: 69 parts, among them Q1 DMG341, SW1 JS102011SAQN, U1 AP7332-3333W6-7SOT23, U2 MCP73831T-2ACI/OT, U3 ATSAMD51G18A-MUT, U4 2MB Flash, U5 REG710NA-5/3K

Commit message: new pycorder and sensor watch
Parts:
- removed R15, R16: 1M, EXB2HV470JV:EXB-2HV470JV
- removed U$32: MATRIX_PASSIVE_8X4SEG, My Stuff:MATRIX_PASSIVE_8X4SEG
- added B1, B2: EVQQ, microbuilder:SWITCH_TACT_SMT_6MM
- added U$24: K1-5202UA, K1-5202UA:K1-5202UA
Connections:
- removed net SWCLK/DISP: C18.1, FFC.DISP, R14.1, TP3.P$1, U3A.PA30/I14/SERCOM1.2/SWCLK/PTCX19+Y19
- removed net SWDIO/EXTCOMIN: FFC.EXTCOMIN, TP6.P$1, U3A.PA31/I15/SERCOM1.3/SWDIO
- removed net X0: R16H.2, U$32.X0Y0, U$32.X0Y1, U$32.X0Y2, U$32.X0Y3, U$32.X0Y4, U3A.PA21/I5/SERCOM3+5.3/I2SDO/PTCX15+Y15
- removed net X1: R16C.2, U$32.X1Y0, U$32.X1Y1, U$32.X1Y2, U$32.X1Y3, U$32.X1Y4, U3A.PA19/I3/SERCOM1+3.3/PTCX13+Y13
- removed net X2: R16B.2, U$32.X2Y0, U$32.X2Y1, U$32.X2Y2, U$32.X2Y3, U$32.X2Y4, U3A.PA18/I2/SERCOM1+3.2//PTCX12+Y12
- removed net X3: R16A.2, U$32.X3Y0, U$32.X3Y1, U$32.X3Y2, U$32.X3Y3, U$32.X3Y4, U3A.PA17/I2C/I1/SERCOM1.1+3.0/PTCX11+Y11
- removed net X4: R15A.2, U$32.X4Y0, U$32.X4Y1, U$32.X4Y2, U$32.X4Y3, U$32.X4Y4, U3A.PA16/I2C/I0/SERCOM1.0+3.1/PTCX10+Y10
- removed net X5: R15B.2, U$32.X5Y0, U$32.X5Y1, U$32.X5Y2, U$32.X5Y3, U$32.X5Y4, U3A.PA15/I15/SERCOM2+4.3
- removed net X6: R15C.2, U$32.X6Y0, U$32.X6Y1, U$32.X6Y2, U$32.X6Y3, U$32.X6Y4, U3A.PA14/I14/SERCOM2+4.2
- removed net X7: R15H.2, U$32.X7Y0, U$32.X7Y1, U$32.X7Y2, U$32.X7Y3, U$32.X7Y4, U3A.PA00/EINT0/SERCOM1.0
- removed net X8: R15G.2, U$32.X8Y0, U$32.X8Y1, U$32.X8Y2, U$32.X8Y3, U$32.X8Y4, U3A.PA01/EINT1/SERCOM1.1
- removed net X9: R15F.2, U$32.X9Y0, U$32.X9Y1, U$32.X9Y2, U$32.X9Y3, U$32.X9Y4, U3A.PA03/I3/VREFA/AIN1/PTCX0+Y0
- removed net Y0: R16G.2, U$32.Y0X0, U$32.Y0X1, U$32.Y0X10, U$32.Y0X2, U$32.Y0X3, U$32.Y0X4, U$32.Y0X5, U$32.Y0X6, U$32.Y0X7, U$32.Y0X8, U$32.Y0X9, U3A.PA20/I4/SERCOM3+5.2/I2SFS0/PTCX14+Y14
- removed net Y1: R16F.2, U$32.Y1X0, U$32.Y1X1, U$32.Y1X10, U$32.Y1X2, U$32.Y1X3, U$32.Y1X4, U$32.Y1X5, U$32.Y1X6, U$32.Y1X7, U$32.Y1X8, U$32.Y1X9, U3A.PA22/I2C/16/SERCOM3.0+5.1/I2SDI/PTCX16+Y16
- removed net Y2: R16E.2, U$32.Y2X0, U$32.Y2X1, U$32.Y2X10, U$32.Y2X2, U$32.Y2X3, U$32.Y2X4, U$32.Y2X5, U$32.Y2X6, U$32.Y2X7, U$32.Y2X8, U$32.Y2X9, U3A.PA23/I2C/I7/SERCOM3.1+5.0/SOF/I2SFS1/PTCX17+Y17
- removed net Y3: R16D.2, U$32.Y3X0, U$32.Y3X1, U$32.Y3X10, U$32.Y3X2, U$32.Y3X3, U$32.Y3X4, U$32.Y3X5, U$32.Y3X6, U$32.Y3X7, U$32.Y3X8, U$32.Y3X9, U3A.PA27/I11/PTCX18+Y18
- new net CENTER: U$24.CENTER, U3A.PA18/I2/SERCOM1+3.2//PTCX12+Y12
- new net DISP: C18.1, FFC.DISP, R14.1, U3A.PA00/EINT0/SERCOM1.0
- new net EXTCOMIN: FFC.EXTCOMIN, U3A.PA01/EINT1/SERCOM1.1
- new net NE: U$24.NE, U3A.PA16/I2C/I0/SERCOM1.0+3.1/PTCX10+Y10
- new net NEXT: B2.S, U3A.PA15/I15/SERCOM2+4.3
- new net NW: U$24.NW, U3A.PA17/I2C/I1/SERCOM1.1+3.0/PTCX11+Y11
- new net PREV: B1.S1, U3A.PA21/I5/SERCOM3+5.3/I2SDO/PTCX15+Y15
- new net SE: U$24.SE, U3A.PA20/I4/SERCOM3+5.2/I2SFS0/PTCX14+Y14
- new net SW: U$24.SW, U3A.PA19/I3/SERCOM1+3.3/PTCX13+Y13
- new net SWCLK: TP3.P$1, U3A.PA30/I14/SERCOM1.2/SWCLK/PTCX19+Y19
- new net SWDIO: TP6.P$1, U3A.PA31/I15/SERCOM1.3/SWDIO
- net 3.3V: now also U3A.PA03/I3/VREFA/AIN1/PTCX0+Y0; no longer R14.2
- net GND: now also B1.P, B1.P1, B2.P, B2.P1, R14.2, U$24.COM, U$24.MP; no longer R15A.1, R15B.1, R15C.1, R15D.1, R15E.1, R15F.1, R15G.1, R15H.1, R16A.1, R16B.1, R16C.1, R16D.1, R16E.1, R16F.1, R16G.1, R16H.1
Other:
- moved on the sheet: R14, TP3, TP6
